Commit message: feat: 로봇 모델을 4바퀴로 다시 변경

File: src/p31/textures/material.xacro (robot description, xacro)
@@ -37,4 +37,13 @@
 		</visual>
 	</gazebo>
+	<gazebo reference="suspension4">
+		<visual>
+				<material>
+					<ambient>${255/255} ${187/255} ${0/255} 1</ambient>
+					<diffuse>${255/255} ${187/255} ${0/255} 1</diffuse>
+					<specular>${255/255} ${187/255} ${0/255} 1</specular>
+				</material>
+		</visual>
+	</gazebo>
 	<gazebo reference="wheel1">
 		<visual>
@@ -45,11 +54,11 @@
 				</material>
 		</visual>
-		<mu1>20.0</mu1>
-		<mu2>40.0</mu2>
+		<mu1>1</mu1>
+		<mu2>1.0</mu2>
 		<kp>500000.0</kp>
 		<kd>10.0</kd>
 		<minDepth>0.001</minDepth>
 		<maxVel>0.1</maxVel>
-		<fdir1>1 0 0</fdir1>
+		<fdir1>0 1 0</fdir1>
 	</gazebo>
 	<gazebo reference="wheel2">
@@ -61,11 +70,11 @@
 				</material>
 		</visual>
-		<mu1>20.0</mu1>
-		<mu2>40.0</mu2>
+		<mu1>1.0</mu1>
+		<mu2>1.0</mu2>
 		<kp>500000.0</kp>
 		<kd>10.0</kd>
 		<minDepth>0.001</minDepth>
 		<maxVel>0.1</maxVel>
-		<fdir1>1 0 0</fdir1>
+		<fdir1>0 1 0</fdir1>
 	</gazebo>
 	<gazebo reference="wheel3">
@@ -77,6 +86,22 @@
 				</material>
 		</visual>
-		<mu1>0.01</mu1>
-		<mu2>0.01</mu2>
+		<mu1>1</mu1>
+		<mu2>1</mu2>
+		<kp>500000.0</kp>
+		<kd>10.0</kd>
+		<minDepth>0.001</minDepth>
+		<maxVel>0.1</maxVel>
+		<fdir1>1 0 0</fdir1>
+	</gazebo>
+	<gazebo reference="wheel4">
+		<visual>
+				<material>
+					<ambient>${5/255} ${0/255} ${153/255} 0.5</ambient>
+					<diffuse>${5/255} ${0/255} ${153/255} 0.5</diffuse>
+					<specular>${5/255} ${0/255} ${153/255} 0.5</specular>
+				</material>
+		</visual>
+		<mu1>1</mu1>
+		<mu2>1</mu2>
 		<kp>500000.0</kp>
 		<kd>10.0</kd>

File: src/p31/urdf/p31.urdf (robot description, URDF)
Before this commit: robot myrobot, 21 links, 20 joints
Links:
- added link suspension4, mass 0.102867975835406; collision mesh filename=package://p31/meshes/suspension2.STL; visual mesh filename=package://p31/meshes/suspension2.STL
- added link wheel4, mass 0.23655; collision cylinder length=0.03 radius=${0.149/2}; visual mesh filename=package://p31/meshes/wheel2.STL
- link suspension3: mass 0.00235619449019234 -> 0.102867975835406; geometry collision mesh filename=package://p31/meshes/suspension1.STL; visual mesh filename=package://p31/meshes/suspension1.STL
- link wheel1: geometry collision cylinder length=0.03 radius=${0.149/2}; visual mesh filename=package://p31/meshes/wheel1.STL
- link wheel2: geometry collision cylinder length=0.03 radius=${0.149/2}; visual mesh filename=package://p31/meshes/wheel2.STL
- link wheel3: mass 0.14667 -> 0.23655; geometry collision cylinder length=0.03 radius=${0.149/2}; visual mesh filename=package://p31/meshes/wheel1.STL
Joints:
- added joint suspension_joint4: type prismatic, parent base_link, child suspension4, origin xyz=-0.135 ${-0.09+0.18} 0.080496 rpy=3.1416 0 1.5708, axis 0 0 1, limit lower=-0.05 upper=0.05 effort=10000 velocity=100000
- added joint wheel_joint4: type continuous, parent suspension4, child wheel4, origin xyz=-0.0133 -0.043 ${-0.00020079-0.00041} rpy=3.1416 1.5708 0, axis 0 -1 0, limit effort=3.1 velocity=7
- joint lidar_joint: origin xyz=-0.00053 -0.10606 ${0.25173+0.03} rpy=0 0 0 -> xyz=-0.00053 -0.10606 ${0.25173+0.03} rpy=0 0 3.141592
- joint suspension_joint3: axis 0 -1 0 -> 0 0 1; origin xyz=0 0.175 0.069998 rpy=1.5708 0 0 -> xyz=0.135 ${-0.09+0.18} 0.080496 rpy=-3.1416 0 1.5708
- joint wheel_joint3: axis 0.028585 -0.036618 0.99892 -> 0 1 0; limit (none) -> effort=3.1 velocity=7; origin xyz=0 -0.032113 0 rpy=-0.036641 -0.028589 -0.23329 -> xyz=-0.0133 0.043 0.00020079 rpy=0 0.5236 0; type fixed -> continuous
