Commit message: change sensor and sources

File: src/p31/urdf/p31.urdf (robot description, URDF)
Before this commit: robot myrobot, 21 links, 20 joints
Joints:
- joint camera_joint2: origin xyz=0.0 -0.08228 ${0.19695} rpy=0 1.5707 -1.5707 -> xyz=0.0 -0.12978 ${0.19695} rpy=0 1.5707 -1.5707
- joint imu_joint: origin xyz=-0.00053 -0.00579 0.25173 rpy=0 0 0 -> xyz=-0.00053 ${0.01341-0.1} 0.25173 rpy=0 0 0
- joint lidar_joint: origin xyz=-0.00053 -0.00579 ${0.25173+0.03} rpy=0 0 0 -> xyz=-0.00053 -0.10606 ${0.25173+0.03} rpy=0 0 0

Commit message: suspension added

File: src/p31/urdf/p31.urdf (robot description, URDF)
Before this commit: robot myrobot, 21 links, 20 joints
Joints:
- joint suspension_joint1: limit lower=0 upper=0.1 effort=0 velocity=0 -> lower=-0.05 upper=0.05 effort=10000 velocity=100000
- joint suspension_joint2: limit lower=0 upper=0.1 effort=0 velocity=0 -> lower=-0.05 upper=0.05 effort=10000 velocity=100000
- joint suspension_joint3: limit lower=0 upper=0.1 effort=0 velocity=0 -> lower=-0.05 upper=0.05 effort=10000 velocity=100000

Commit message: imu and lidar position changed

File: src/p31/urdf/p31.urdf (robot description, URDF)
Before this commit: robot myrobot, 23 links, 22 joints
Joints:
- joint imu_joint: origin xyz=-0.00053 ${0.01341-0.1} 0.25173 rpy=0 0 0 -> xyz=-0.00053 0 0.25173 rpy=0 0 0
- joint lidar_joint: origin xyz=-0.00053 -0.10606 ${0.25173+0.03} rpy=0 0 3.141592 -> xyz=-0.00053 0 ${0.25173+0.03} rpy=0 0 3.141592

Commit message: feat: Add test IMU and update C,K values

File: src/p31/urdf/p31.urdf (robot description, URDF)
Before this commit: robot myrobot, 23 links, 22 joints
Links:
- added link imu_test; visual cylinder length=0.02 radius=0.01
Joints:
- added joint imu_test_joint: type fixed, parent base_link, child imu_link, origin xyz=-0.00053 0 0.25173 rpy=0 0 0

File: src/p31/urdf/sensor.gazebo.xacro (robot description, xacro)
@@ -46,4 +46,38 @@
       <frameName>imu_link</frameName>
       <topicName>imu</topicName>
+      <serviceName>imu_service</serviceName>
+      <gaussianNoise>0.0</gaussianNoise>
+      <updateRate>200</updateRate>
+      <imu>
+        <noise>
+          <type>gaussian</type>
+          <rate>
+            <mean>0.0</mean>
+            <stddev>2e-4</stddev>
+            <bias_mean>0.0000075</bias_mean>
+            <bias_stddev>0.0000008</bias_stddev>
+          </rate>
+          <accel>
+            <mean>0.0</mean>
+            <stddev>1.7e-2</stddev>
+            <bias_mean>0.1</bias_mean>
+            <bias_stddev>0.001</bias_stddev>
+          </accel>
+        </noise>
+      </imu>
+    </plugin>
+  </gazebo>
+  <gazebo reference="imu_test">
+    <sensor type="imu" name="imu">
+      <always_on>true</always_on>
+    </sensor>
+    <material>Gazebo/Grey</material>
+  </gazebo>
+   <gazebo>
+    <plugin name="imu_plugin" filename="libgazebo_ros_imu.so">
+      <alwaysOn>true</alwaysOn>
+      <bodyName>imu_test</bodyName>
+      <frameName>imu_test</frameName>
+      <topicName>imu_test</topicName>
       <serviceName>imu_service</serviceName>
       <gaussianNoise>0.0</gaussianNoise>

Commit message: last minute fixes

File: src/p31/urdf/p31.urdf (robot description, URDF)
Before this commit: robot myrobot, 24 links, 23 joints
Joints:
- joint imu_test_joint: child imu_link -> imu_test

File: src/p31/urdf/sensor.gazebo.xacro (robot description, xacro)
@@ -69,5 +69,5 @@
   </gazebo>
   <gazebo reference="imu_test">
-    <sensor type="imu" name="imu">
+    <sensor type="imu" name="imu_test">
       <always_on>true</always_on>
     </sensor>
@@ -80,6 +80,6 @@
       <frameName>imu_test</frameName>
       <topicName>imu_test</topicName>
-      <serviceName>imu_service</serviceName>
-      <gaussianNoise>0.0</gaussianNoise>
+      <serviceName>imu_service_test</serviceName>
+      <gaussianNoise>0.1</gaussianNoise>
       <updateRate>200</updateRate>
       <imu>
